Commit message: dual urdf fix

File: dual_ur_robotiq_description/urdf/robot.urdf.xacro (robot description, xacro)
@@ -8,9 +8,11 @@
     <inertial>
         <mass value="1000" />
-        <origin xyz="0 0 1.8" rpy="0 0 ${PI/2}" />
+        <!--<origin xyz="0 0 1.8" rpy="0 0 ${PI/2}" />-->
+        <origin rpy="0 0 ${PI/2}" xyz="0 0 1.57"/>
         <inertia ixx="0.01" ixy="0" ixz="0" iyy="0.01" iyz="0" izz="0.01" />
     </inertial>
     <visual>
-      <origin xyz="0 0 1.8" rpy="0 0 ${PI/2}"/>
+     <!-- <origin xyz="0 0 1.8" rpy="0 0 ${PI/2}"/>-->
+     <origin rpy="0 0 ${PI/2}" xyz="0 0 1.57"/>
       <geometry>
         <mesh filename="package://dual_ur_robotiq_description/meshes/dual_arm_mount.stl" scale="0.03 0.03 0.03" />
@@ -21,5 +23,6 @@
     </visual>
     <collision>
-      <origin xyz="0 0 1.8" rpy="0 0 ${PI/2}"/>
+      <!--<origin xyz="0 0 1.8" rpy="0 0 ${PI/2}"/>-->
+      <origin rpy="0 0 ${PI/2}" xyz="0 0 1.57"/>
       <geometry>
         <mesh filename="package://dual_ur_robotiq_description/meshes/dual_arm_mount.stl" scale="0.03 0.03 0.03" />
@@ -47,5 +50,6 @@
     <child link = "right_base_link" />
     <!--origin xyz="0 0.3 1.8" rpy="${PI/4*3} 0.028 ${PI}" /-->
-    <origin xyz="0 0.305 1.65" rpy="${PI/4*3} 0 ${PI}" />
+    <!--<origin xyz="0 0.305 1.65" rpy="${PI/4*3} 0 ${PI}" />-->
+    <origin rpy="${PI/4*3} 0 ${PI}" xyz="0 0.305 1.56"/>
   </joint>
   <joint name="left_arm_joint" type="fixed">
@@ -53,5 +57,6 @@
     <child link = "left_base_link" />
     <!--origin xyz="0 -0.3 1.803" rpy="${(PI/4*3)+0.003} -0.005 0" /-->
-    <origin xyz="-0.01 -0.305 1.65" rpy="${PI/4*3} 0 0" />
+    <!--<origin xyz="-0.01 -0.305 1.65" rpy="${PI/4*3} 0 0" />-->
+    <origin rpy="${PI/4*3} 0 0" xyz="-0.01 -0.305 1.56"/>
     <!-- origin xyz="0 -0.3 1.65" rpy="${PI/4*3} 0 0" /-->
   </joint>
